File: Schematics/Rocket Control Board/Rocket-Control.sch (EAGLE design)
At the start: 37 parts

Commit message: Rocket Control Board Work
Significant changes to rocket control board. Too many to detail.
Parts:
- removed U$11, U$12, U$13, U$14, U$15, U$16, U$17, U$18, U$19, U$20, U$23, U$24, U$25, U$27, U$28, U$29, U$30, U$31, U$32, U$33, U$34, U$36, U$37, U$5: HEADER-HOLE, RocketControlBoard:HEADER-HOLE
- added U$38: 10118194-0001LF:MICRO-USB, RocketControlBoard:10118194-0001LF:MICRO-USB
- added U$41: SPI-PORT, RocketControlBoard:SPI-PORT
- added U$56: VDDCORE-CAPACITOR, RocketControlBoard:VDDCORE-CAPACITOR
- added U$57: VIN-CAPACITOR, RocketControlBoard:VIN-CAPACITOR
- added U$61: JTAG-MINI, RocketControlBoard:JTAG-MINI
- U$21: value HEADER-HOLE -> HEADER-SIDE-A; device RocketControlBoard:HEADER-HOLE -> RocketControlBoard:HEADER-SIDE-A
- U$22: value HEADER-HOLE -> HEADER-SIDE-B; device RocketControlBoard:HEADER-HOLE -> RocketControlBoard:HEADER-SIDE-B
Connections:
- new net A5: U$1.PB02:ANALOG-A5, U$21.A5
- new net RX: U$1.PB23:RX
- new net SWD-06(RESET): U$1.--RESET:BUTTON+SWD-06, U$61.RESET
- new net SWD-09: U$1.PA30:SWD-09, U$61.JTAG09
- new net SWD-10: U$1.PA31:SWD-10, U$61.JTAG10
- new net TX: U$1.PB22:TX
- new net USB: U$22.USB, U$38.5V
- new net VDDCORE: U$1.VDDCORE:GND, U$56.P$1
- new net VIN: U$1.VDDIN:VIN, U$22.VIN, U$57.P$1
- net +3V3: now also U$22.3V3, U$41.VIN, U$61.VIN; no longer U$36.HOLE
- net A0: now also U$21.A0; no longer U$5.HOLE
- net A1: now also U$21.A1; no longer U$11.HOLE
- net A2: now also U$21.A2; no longer U$12.HOLE
- net A3: now also U$21.A3; no longer U$13.HOLE
- net A4: now also U$21.A4; no longer U$14.HOLE
- net AREF: now also U$21.AREF
- net D0-TX: now also U$21.D0; no longer U$18.HOLE
- net D1-RX: now also U$21.D1; no longer U$17.HOLE
- net D10: now also U$22.10; no longer U$30.HOLE
- net D11: now also U$22.11; no longer U$32.HOLE
- net D12: now also U$22.12; no longer U$29.HOLE
- net D13: now also U$22.13; no longer U$31.HOLE
- net D2: now also U$21.D2; no longer U$20.HOLE
- net D3: now also U$21.D3; no longer U$19.HOLE
- net D4: now also U$21.D4; no longer U$24.HOLE
- net D5: now also U$21.D5; no longer U$25.HOLE
- net D6: now also U$21.D6; no longer U$28.HOLE
- net D7: now also U$22.7, U$41.ATN; no longer U$27.HOLE
- net D8: now also U$22.8; no longer U$15.HOLE
- net D9: now also U$22.9; no longer U$16.HOLE
- net GND: now also U$1.GND:GND, U$22.GND-IN, U$22.GND-OUT, U$38.GND, U$41.GND, U$56.P$2, U$57.P$2, U$61.GND-1, U$61.GND-2, U$61.GND-3; no longer U$37.HOLE
- net MISO: now also U$41.MISO; no longer U$23.HOLE
- net MOSI: now also U$41.MOSI; no longer U$21.HOLE
- net SCK: now also U$41.SCK; no longer U$22.HOLE
- net SCL: now also U$22.SCL; no longer U$34.HOLE
- net SDA: now also U$22.SDA; no longer U$33.HOLE
- net USB-N: now also U$38.D-
- net USB-P: now also U$38.D+

Commit message: Added Regulator Part
See Title
Parts:
- added U$5: REGULATOR, RocketControlBoard:REGULATOR
Connections:
- new net VIN-REGULATED: U$1.VDDIN:VIN, U$57.P$1
- net VIN: no longer U$1.VDDIN:VIN, U$57.P$1
Changed lines of the file:
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@@
 <part name="U$21" library="RocketControlBoard" deviceset="HEADER-SIDE-A" device=""/>
 <part name="U$22" library="RocketControlBoard" deviceset="HEADER-SIDE-B" device=""/>
+<part name="U$5" library="RocketControlBoard" deviceset="REGULATOR" device=""/>
 </parts>
 <sheets>
@@
 <instance part="U$21" gate="G$1" x="48.26" y="-40.64" rot="R180"/>
 <instance part="U$22" gate="G$1" x="104.14" y="-40.64" rot="R180"/>
+<instance part="U$5" gate="G$1" x="-33.02" y="-50.8"/>
 </instances>
 <busses>
@@
 <segment>
 <pinref part="U$56" gate="G$1" pin="P$1"/>
-<wire x1="185.42" y1="35.56" x2="175.26" y2="35.56" width="0.1524" layer="91"/>
-<label x="175.26" y="35.56" size="1.778" layer="95"/>
+<wire x1="185.42" y1="35.56" x2="167.64" y2="35.56" width="0.1524" layer="91"/>
+<label x="167.64" y="35.56" size="1.778" layer="95"/>
 </segment>
 </net>
 <net name="VIN" class="0">
+<segment>
+<wire x1="109.22" y1="-40.64" x2="104.14" y2="-40.64" width="0.1524" layer="91"/>
+<pinref part="U$22" gate="G$1" pin="VIN"/>
+<label x="109.22" y="-40.64" size="1.778" layer="95"/>
+</segment>
+</net>
+<net name="A5" class="0">
+<segment>
+<pinref part="U$1" gate="G$1" pin="PB02:ANALOG-A5"/>
+<wire x1="111.76" y1="66.04" x2="121.92" y2="66.04" width="0.1524" layer="91"/>
+<label x="124.46" y="66.04" size="1.778" layer="95"/>
+</segment>
+<segment>
+<wire x1="58.42" y1="-25.4" x2="53.34" y2="-25.4" width="0.1524" layer="91"/>
+<pinref part="U$21" gate="G$1" pin="A5"/>
+<label x="58.42" y="-25.4" size="1.778" layer="95"/>
+</segment>
+</net>
+<net name="SWD-10" class="0">
+<segment>
+<pinref part="U$1" gate="G$1" pin="PA31:SWD-10"/>
+<wire x1="111.76" y1="63.5" x2="121.92" y2="63.5" width="0.1524" layer="91"/>
+<label x="124.46" y="63.5" size="1.778" layer="95"/>
+</segment>
+<segment>
+<pinref part="U$61" gate="G$1" pin="JTAG10"/>
+<wire x1="210.82" y1="109.22" x2="223.52" y2="109.22" width="0.1524" layer="91"/>
+<label x="218.44" y="109.22" size="1.778" layer="95"/>
+</segment>
+</net>
+<net name="SWD-09" class="0">
+<segment>
+<pinref part="U$1" gate="G$1" pin="PA30:SWD-09"/>
+<wire x1="111.76" y1="60.96" x2="121.92" y2="60.96" width="0.1524" layer="91"/>
+<label x="124.46" y="60.96" size="1.778" layer="95"/>
+</segment>
+<segment>
+<pinref part="U$61" gate="G$1" pin="JTAG09"/>
+<wire x1="223.52" y1="106.68" x2="210.82" y2="106.68" width="0.1524" layer="91"/>
+<label x="218.44" y="106.68" size="1.778" layer="95"/>
+</segment>
+</net>
+<net name="TX" class="0">
+<segment>
+<pinref part="U$1" gate="G$1" pin="PB22:TX"/>
+<wire x1="111.76" y1="40.64" x2="121.92" y2="40.64" width="0.1524" layer="91"/>
+<label x="124.46" y="40.64" size="1.778" layer="95"/>
+</segment>
+</net>
+<net name="VIN-REGULATED" class="0">
 <segment>
 <pinref part="U$1" gate="G$1" pin="VDDIN:VIN"/>
@@
 </segment>
 <segment>
-<wire x1="175.26" y1="55.88" x2="185.42" y2="55.88" width="0.1524" layer="91"/>
-<label x="175.26" y="55.88" size="1.778" layer="95"/>
+<wire x1="167.64" y1="55.88" x2="185.42" y2="55.88" width="0.1524" layer="91"/>
+<label x="167.64" y="55.88" size="1.778" layer="95"/>
 <pinref part="U$57" gate="G$1" pin="P$1"/>
 </segment>
-<segment>
-<wire x1="109.22" y1="-40.64" x2="104.14" y2="-40.64" width="0.1524" layer="91"/>
-<pinref part="U$22" gate="G$1" pin="VIN"/>
-<label x="109.22" y="-40.64" size="1.778" layer="95"/>
-</segment>
-</net>
-<net name="A5" class="0">
-<segment>
-<pinref part="U$1" gate="G$1" pin="PB02:ANALOG-A5"/>
-<wire x1="111.76" y1="66.04" x2="121.92" y2="66.04" width="0.1524" layer="91"/>
-<label x="124.46" y="66.04" size="1.778" layer="95"/>
-</segment>
-<segment>
-<wire x1="58.42" y1="-25.4" x2="53.34" y2="-25.4" width="0.1524" layer="91"/>
-<pinref part="U$21" gate="G$1" pin="A5"/>
-<label x="58.42" y="-25.4" size="1.778" layer="95"/>
-</segment>
-</net>
-<net name="SWD-10" class="0">
-<segment>
-<pinref part="U$1" gate="G$1" pin="PA31:SWD-10"/>
-<wire x1="111.76" y1="63.5" x2="121.92" y2="63.5" width="0.1524" layer="91"/>
-<label x="124.46" y="63.5" size="1.778" layer="95"/>
-</segment>
-<segment>
-<pinref part="U$61" gate="G$1" pin="JTAG10"/>
-<wire x1="210.82" y1="109.22" x2="223.52" y2="109.22" width="0.1524" layer="91"/>
-<label x="218.44" y="109.22" size="1.778" layer="95"/>
-</segment>
-</net>
-<net name="SWD-09" class="0">
-<segment>
-<pinref part="U$1" gate="G$1" pin="PA30:SWD-09"/>
-<wire x1="111.76" y1="60.96" x2="121.92" y2="60.96" width="0.1524" layer="91"/>
-<label x="124.46" y="60.96" size="1.778" layer="95"/>
-</segment>
-<segment>
-<pinref part="U$61" gate="G$1" pin="JTAG09"/>
-<wire x1="223.52" y1="106.68" x2="210.82" y2="106.68" width="0.1524" layer="91"/>
-<label x="218.44" y="106.68" size="1.778" layer="95"/>
-</segment>
-</net>
-<net name="TX" class="0">
-<segment>
-<pinref part="U$1" gate="G$1" pin="PB22:TX"/>
-<wire x1="111.76" y1="40.64" x2="121.92" y2="40.64" width="0.1524" layer="91"/>
-<label x="124.46" y="40.64" size="1.778" layer="95"/>
-</segment>
-</net>
+</net>

Commit message: Added regulator and supporting components
Parts:
- added U$11, U$12: REGULATOR-CAPACITORS, RocketControlBoard:REGULATOR-CAPACITORS
- added U$13: REGULATOR-INDUCTOR, RocketControlBoard:REGULATOR-INDUCTOR
- added U$14: REGULATOR-RESISTOR, RocketControlBoard:REGULATOR-RESISTOR
Connections:
- new net N$1: U$13.P$1, U$5.PG
- new net N$3: U$14.P$1, U$5.VOS
- net GND: now also U$11.A, U$12.A, U$5.AGND, U$5.EN, U$5.ETP, U$5.FB
- net VIN: now also U$11.B, U$5.PGND, U$5.VIN
- net VIN-REGULATED: now also U$12.B, U$13.P$2, U$14.P$2, U$5.SW
Changed lines of the file:
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@@
 <part name="U$22" library="RocketControlBoard" deviceset="HEADER-SIDE-B" device=""/>
 <part name="U$5" library="RocketControlBoard" deviceset="REGULATOR" device=""/>
+<part name="U$11" library="RocketControlBoard" deviceset="REGULATOR-CAPACITORS" device=""/>
+<part name="U$12" library="RocketControlBoard" deviceset="REGULATOR-CAPACITORS" device=""/>
+<part name="U$13" library="RocketControlBoard" deviceset="REGULATOR-INDUCTOR" device=""/>
+<part name="U$14" library="RocketControlBoard" deviceset="REGULATOR-RESISTOR" device=""/>
+<part name="GND10" library="supply1" deviceset="GND" device=""/>
+<part name="GND11" library="supply1" deviceset="GND" device=""/>
+<part name="GND16" library="supply1" deviceset="GND" device=""/>
 </parts>
 <sheets>
@@
 <instance part="U$21" gate="G$1" x="48.26" y="-40.64" rot="R180"/>
 <instance part="U$22" gate="G$1" x="104.14" y="-40.64" rot="R180"/>
-<instance part="U$5" gate="G$1" x="-33.02" y="-50.8"/>
+<instance part="U$5" gate="G$1" x="-60.96" y="-45.72"/>
+<instance part="U$11" gate="G$1" x="-96.52" y="-48.26" rot="R90"/>
+<instance part="U$12" gate="G$1" x="2.54" y="-55.88" rot="R90"/>
+<instance part="U$13" gate="G$1" x="-25.4" y="-40.64"/>
+<instance part="U$14" gate="G$1" x="-10.16" y="-55.88" rot="R90"/>
+<instance part="GND10" gate="1" x="-96.52" y="-63.5"/>
+<instance part="GND11" gate="1" x="2.54" y="-73.66"/>
+<instance part="GND16" gate="1" x="-60.96" y="-63.5"/>
 </instances>
 <busses>
@@
 <pinref part="U$22" gate="G$1" pin="GND-IN"/>
 <label x="109.22" y="-38.1" size="1.778" layer="95"/>
+</segment>
+<segment>
+<pinref part="U$5" gate="G$1" pin="AGND"/>
+<wire x1="-76.2" y1="-50.8" x2="-81.28" y2="-50.8" width="0.1524" layer="91"/>
+<wire x1="-81.28" y1="-50.8" x2="-88.9" y2="-50.8" width="0.1524" layer="91"/>
+<wire x1="-88.9" y1="-50.8" x2="-88.9" y2="-60.96" width="0.1524" layer="91"/>
+<pinref part="U$11" gate="G$1" pin="A"/>
+<wire x1="-88.9" y1="-60.96" x2="-96.52" y2="-60.96" width="0.1524" layer="91"/>
+<pinref part="U$5" gate="G$1" pin="EN"/>
+<wire x1="-76.2" y1="-48.26" x2="-81.28" y2="-48.26" width="0.1524" layer="91"/>
+<wire x1="-81.28" y1="-48.26" x2="-81.28" y2="-50.8" width="0.1524" layer="91"/>
+<wire x1="-96.52" y1="-60.96" x2="-106.68" y2="-60.96" width="0.1524" layer="91"/>
+<pinref part="GND10" gate="1" pin="GND"/>
+<junction x="-96.52" y="-60.96"/>
+<label x="-111.76" y="-60.96" size="1.778" layer="95"/>
+</segment>
+<segment>
+<pinref part="U$5" gate="G$1" pin="FB"/>
+<wire x1="-45.72" y1="-50.8" x2="-40.64" y2="-50.8" width="0.1524" layer="91"/>
+<wire x1="-40.64" y1="-50.8" x2="-40.64" y2="-71.12" width="0.1524" layer="91"/>
+<pinref part="U$12" gate="G$1" pin="A"/>
+<wire x1="-40.64" y1="-71.12" x2="2.54" y2="-71.12" width="0.1524" layer="91"/>
+<wire x1="2.54" y1="-71.12" x2="2.54" y2="-68.58" width="0.1524" layer="91"/>
+<wire x1="2.54" y1="-71.12" x2="10.16" y2="-71.12" width="0.1524" layer="91"/>
+<pinref part="GND11" gate="1" pin="GND"/>
+<junction x="2.54" y="-71.12"/>
+<label x="10.16" y="-71.12" size="1.778" layer="95"/>
+</segment>
+<segment>
+<pinref part="U$5" gate="G$1" pin="ETP"/>
+<pinref part="GND16" gate="1" pin="GND"/>
 </segment>
 </net>
@@
 <label x="109.22" y="-40.64" size="1.778" layer="95"/>
 </segment>
+<segment>
+<pinref part="U$5" gate="G$1" pin="PGND"/>
+<wire x1="-76.2" y1="-43.18" x2="-81.28" y2="-43.18" width="0.1524" layer="91"/>
+<wire x1="-81.28" y1="-43.18" x2="-88.9" y2="-43.18" width="0.1524" layer="91"/>
+<wire x1="-88.9" y1="-43.18" x2="-88.9" y2="-35.56" width="0.1524" layer="91"/>
+<pinref part="U$11" gate="G$1" pin="B"/>
+<wire x1="-88.9" y1="-35.56" x2="-96.52" y2="-35.56" width="0.1524" layer="91"/>
+<pinref part="U$5" gate="G$1" pin="VIN"/>
+<wire x1="-76.2" y1="-45.72" x2="-81.28" y2="-45.72" width="0.1524" layer="91"/>
+<wire x1="-81.28" y1="-45.72" x2="-81.28" y2="-43.18" width="0.1524" layer="91"/>
+<wire x1="-96.52" y1="-35.56" x2="-106.68" y2="-35.56" width="0.1524" layer="91"/>
+<label x="-111.76" y="-35.56" size="1.778" layer="95"/>
+</segment>
 </net>
 <net name="A5" class="0">
@@
 <pinref part="U$57" gate="G$1" pin="P$1"/>
 </segment>
-</net>
+<segment>
+<pinref part="U$13" gate="G$1" pin="P$2"/>
+<pinref part="U$14" gate="G$1" pin="P$2"/>
+<wire x1="-12.7" y1="-40.64" x2="-10.16" y2="-40.64" width="0.1524" layer="91"/>
+<wire x1="-10.16" y1="-40.64" x2="-10.16" y2="-43.18" width="0.1524" layer="91"/>
+<pinref part="U$12" gate="G$1" pin="B"/>
+<wire x1="-10.16" y1="-40.64" x2="2.54" y2="-40.64" width="0.1524" layer="91"/>
+<wire x1="2.54" y1="-40.64" x2="2.54" y2="-43.18" width="0.1524" layer="91"/>
+<wire x1="2.54" y1="-40.64" x2="10.16" y2="-40.64" width="0.1524" layer="91"/>
+<pinref part="U$5" gate="G$1" pin="SW"/>
+<wire x1="-45.72" y1="-45.72" x2="-15.24" y2="-45.72" width="0.1524" layer="91"/>
+<wire x1="-15.24" y1="-45.72" x2="-10.16" y2="-40.64" width="0.1524" layer="91"/>
+<label x="10.16" y="-40.64" size="1.778" layer="95"/>
+</segment>
+</net>
+<net name="N$1" class="0">
+<segment>
+<pinref part="U$5" gate="G$1" pin="PG"/>
+<pinref part="U$13" gate="G$1" pin="P$1"/>
+<wire x1="-45.72" y1="-43.18" x2="-38.1" y2="-43.18" width="0.1524" layer="91"/>
+<wire x1="-38.1" y1="-43.18" x2="-38.1" y2="-40.64" width="0.1524" layer="91"/>
+</segment>
+</net>
+<net name="N$3" class="0">
+<segment>
+<pinref part="U$14" gate="G$1" pin="P$1"/>
+<wire x1="-10.16" y1="-68.58" x2="-38.1" y2="-68.58" width="0.1524" layer="91"/>
+<wire x1="-38.1" y1="-68.58" x2="-38.1" y2="-48.26" width="0.1524" layer="91"/>
+<pinref part="U$5" gate="G$1" pin="VOS"/>
+<wire x1="-38.1" y1="-48.26" x2="-45.72" y2="-48.26" width="0.1524" layer="91"/>
+</segment>
+</net>

Commit message: Added Diode, Began Routing
Parts:
- added U$15: REGULATION-DIODE, RocketControlBoard:REGULATION-DIODE
Connections:
- net USB: now also U$15.P$1
- net VIN: now also U$15.P$2
Changed lines of the file:
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@@
 <?xml version="1.0" encoding="utf-8"?>
 <!DOCTYPE eagle SYSTEM "eagle.dtd">
-<eagle version="7.5.0">
+<eagle version="7.6.0">
 <drawing>
 <settings>
@@
 <part name="GND11" library="supply1" deviceset="GND" device=""/>
 <part name="GND16" library="supply1" deviceset="GND" device=""/>
+<part name="U$15" library="RocketControlBoard" deviceset="REGULATION-DIODE" device=""/>
 </parts>
 <sheets>
@@
 <instance part="GND11" gate="1" x="2.54" y="-73.66"/>
 <instance part="GND16" gate="1" x="-60.96" y="-63.5"/>
+<instance part="U$15" gate="G$1" x="78.74" y="-71.12"/>
 </instances>
 <busses>
@@
 <label x="109.22" y="-35.56" size="1.778" layer="95"/>
 </segment>
+<segment>
+<pinref part="U$15" gate="G$1" pin="P$1"/>
+<wire x1="66.04" y1="-71.12" x2="50.8" y2="-71.12" width="0.1524" layer="91"/>
+<label x="50.8" y="-71.12" size="1.778" layer="95"/>
+</segment>
 </net>
 <net name="RX" class="0">
@@
 <label x="-111.76" y="-35.56" size="1.778" layer="95"/>
 </segment>
-</net>
+<segment>
+<pinref part="U$15" gate="G$1" pin="P$2"/>
+<wire x1="91.44" y1="-71.12" x2="109.22" y2="-71.12" width="0.1524" layer="91"/>
+<label x="104.14" y="-71.12" size="1.778" layer="95"/>
+</segment>
+</net>

Commit message: Misc Routing
Connections:
- net +3V3: now also U$12.B, U$13.P$2, U$14.P$2, U$5.SW
- net VIN-REGULATED: no longer U$12.B, U$13.P$2, U$14.P$2, U$5.SW
Changed lines of the file:
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@@
 <part name="GND16" library="supply1" deviceset="GND" device=""/>
 <part name="U$15" library="RocketControlBoard" deviceset="REGULATION-DIODE" device=""/>
+<part name="+3V4" library="supply1" deviceset="+3V3" device=""/>
 </parts>
 <sheets>
@@
 <instance part="GND16" gate="1" x="-60.96" y="-63.5"/>
 <instance part="U$15" gate="G$1" x="78.74" y="-71.12"/>
+<instance part="+3V4" gate="G$1" x="2.54" y="-30.48"/>
 </instances>
 <busses>
@@
 <label x="109.22" y="-30.48" size="1.778" layer="95"/>
 </segment>
+<segment>
+<pinref part="U$13" gate="G$1" pin="P$2"/>
+<pinref part="U$14" gate="G$1" pin="P$2"/>
+<wire x1="-12.7" y1="-40.64" x2="-10.16" y2="-40.64" width="0.1524" layer="91"/>
+<wire x1="-10.16" y1="-40.64" x2="-10.16" y2="-43.18" width="0.1524" layer="91"/>
+<pinref part="U$12" gate="G$1" pin="B"/>
+<wire x1="-10.16" y1="-40.64" x2="2.54" y2="-40.64" width="0.1524" layer="91"/>
+<wire x1="2.54" y1="-40.64" x2="2.54" y2="-43.18" width="0.1524" layer="91"/>
+<wire x1="2.54" y1="-40.64" x2="2.54" y2="-33.02" width="0.1524" layer="91"/>
+<pinref part="U$5" gate="G$1" pin="SW"/>
+<wire x1="-45.72" y1="-45.72" x2="-15.24" y2="-45.72" width="0.1524" layer="91"/>
+<wire x1="-15.24" y1="-45.72" x2="-10.16" y2="-40.64" width="0.1524" layer="91"/>
+<pinref part="+3V4" gate="G$1" pin="+3V3"/>
+</segment>
 </net>
 <net name="ANALOG-VDD" class="0">
@@
 <pinref part="U$57" gate="G$1" pin="P$1"/>
 </segment>
-<segment>
-<pinref part="U$13" gate="G$1" pin="P$2"/>
-<pinref part="U$14" gate="G$1" pin="P$2"/>
-<wire x1="-12.7" y1="-40.64" x2="-10.16" y2="-40.64" width="0.1524" layer="91"/>
-<wire x1="-10.16" y1="-40.64" x2="-10.16" y2="-43.18" width="0.1524" layer="91"/>
-<pinref part="U$12" gate="G$1" pin="B"/>
-<wire x1="-10.16" y1="-40.64" x2="2.54" y2="-40.64" width="0.1524" layer="91"/>
-<wire x1="2.54" y1="-40.64" x2="2.54" y2="-43.18" width="0.1524" layer="91"/>
-<wire x1="2.54" y1="-40.64" x2="10.16" y2="-40.64" width="0.1524" layer="91"/>
-<pinref part="U$5" gate="G$1" pin="SW"/>
-<wire x1="-45.72" y1="-45.72" x2="-15.24" y2="-45.72" width="0.1524" layer="91"/>
-<wire x1="-15.24" y1="-45.72" x2="-10.16" y2="-40.64" width="0.1524" layer="91"/>
-<label x="10.16" y="-40.64" size="1.778" layer="95"/>
-</segment>
-</net>
+</net>
