File: Schematics/Rocket Control Board/Version-5/Rocket-Control5.brd (EAGLE design)
At the start: 20.3 x 38.1 mm, 29 parts

Commit message: Final commit for the semester
Various board changes.
Connections:
- net GND: now also U$5.PGND; no longer U$5.EN
- net REG-VIN: now also U$5.EN; no longer U$5.PGND
Routing:
- net D3: track 10.8 -> 4.79 mm
Changed lines of the file:
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@@
 <contactref element="U$22" pad="GND-OUT"/>
 <contactref element="U$22" pad="GND-IN"/>
-<contactref element="U$5" pad="AGND"/>
 <contactref element="U$11" pad="1"/>
-<contactref element="U$5" pad="EN"/>
 <contactref element="U$12" pad="1"/>
 <contactref element="U$5" pad="EXPOSED-THERMAL-PAD"/>
@@
 <wire x1="15.113" y1="20.474446875" x2="15.113" y2="22.1742" width="0.1524" layer="1"/>
 <wire x1="15.113" y1="22.1742" x2="15.9258" y2="22.987" width="0.1524" layer="1"/>
+<contactref element="U$5" pad="AGND"/>
+<contactref element="U$5" pad="PGND"/>
 </signal>
 <signal name="A0">
@@
 <wire x1="15.90738125" y1="18.4404" x2="16.8402" y2="18.4404" width="0.1524" layer="1"/>
 <via x="16.8402" y="18.4404" extent="1-16" drill="0.3302"/>
-<wire x1="16.8402" y1="18.4404" x2="16.8402" y2="24.4602" width="0.1524" layer="16"/>
+<wire x1="16.8402" y1="18.4404" x2="16.8402" y2="24.4602" width="0" layer="19" extent="1-16"/>
 <wire x1="16.8402" y1="24.4602" x2="19.05" y2="26.67" width="0.1524" layer="16"/>
 </signal>
@@
 </signal>
 <signal name="REG-VIN">
-<contactref element="U$5" pad="PGND"/>
 <contactref element="U$11" pad="2"/>
-<contactref element="U$5" pad="VIN"/>
 <contactref element="U$15" pad="P$2"/>
 <contactref element="U$16" pad="P$2"/>
-<wire x1="5.9436" y1="31.2524" x2="6.8914" y2="31.2524" width="0.1524" layer="1"/>
-<wire x1="6.8914" y1="31.2524" x2="7.2898" y2="31.2524" width="0.1524" layer="1"/>
+<wire x1="5.9436" y1="31.2524" x2="7.2898" y2="31.2524" width="0.1524" layer="1"/>
 <wire x1="7.2898" y1="31.2524" x2="7.3914" y2="31.1508" width="0.1524" layer="1"/>
-<wire x1="7.3914" y1="31.1508" x2="7.3914" y2="30.0736" width="0.1524" layer="1"/>
-<wire x1="6.8914" y1="30.0736" x2="6.8914" y2="31.2524" width="0.1524" layer="1"/>
 <wire x1="5.9436" y1="31.2524" x2="4.8214" y2="31.2524" width="0.1524" layer="1"/>
 <wire x1="4.8214" y1="31.2524" x2="4.1656" y2="30.5966" width="0.1524" layer="1"/>
+<contactref element="U$5" pad="VIN"/>
+<contactref element="U$5" pad="EN"/>
+<wire x1="6.8914" y1="30.0736" x2="6.8914" y2="30.854" width="0.1524" layer="1"/>
+<wire x1="6.8914" y1="30.854" x2="7.2898" y2="31.2524" width="0.1524" layer="1"/>
+<wire x1="6.3914" y1="30.0736" x2="6.3914" y2="30.8046" width="0.1524" layer="1"/>
+<wire x1="6.3914" y1="30.8046" x2="5.9436" y2="31.2524" width="0.1524" layer="1"/>
 </signal>
 <signal name="N$2">

Commit message: Version 6
Version 6 of the board
Next blog post
Added ULP Scripts that help make a bill of materials.
Parts:
- added U$23, U$24: HEADER-HOLE, RocketControlBoard:HEADER-HOLE
Connections:
- new net USB-ID-BOARD: U$23.P$1, U$38.4:ID
- new net USB-ID-CHIP: U$1.41, U$24.P$1
Changed lines of the file:
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@@
 <element name="U$19" library="RocketControlBoard" package="C0402" value="I2C-PULLUP" x="4.1656" y="23.749" rot="R270"/>
 <element name="U$20" library="RocketControlBoard" package="C0402" value="I2C-PULLUP" x="4.1656" y="20.6756" rot="R270"/>
+<element name="U$23" library="RocketControlBoard" package="HEADER-HOLE" value="HEADER-HOLE" x="0" y="-2.159"/>
+<element name="U$24" library="RocketControlBoard" package="HEADER-HOLE" value="HEADER-HOLE" x="0" y="-4.2164"/>
 </elements>
 <signals>
@@
 <wire x1="15.963" y1="36.7284" x2="15.963" y2="34.4424" width="0.1524" layer="1"/>
 </signal>
+<signal name="USB-ID-CHIP">
+<contactref element="U$1" pad="41"/>
+<contactref element="U$24" pad="P$1"/>
+<wire x1="0" y1="-4.2164" x2="7.259465625" y2="14.035125" width="0" layer="19" extent="1-1"/>
+</signal>
+<signal name="USB-ID-BOARD">
+<contactref element="U$23" pad="P$1"/>
+<contactref element="U$38" pad="4:ID"/>
+<wire x1="0" y1="-2.159" x2="8.0114" y2="34.0284" width="0" layer="19" extent="1-1"/>
+</signal>
 </signals>
